Commit message: extend baseline to 40cm fix the bug of roi out of range.

File: models/left_camera.xacro (robot description, xacro)
@@ -45,5 +45,5 @@
                         <type>gaussian</type>
                         <mean>0.0</mean>
-                        <stddev>0.007</stddev>
+                        <stddev>0.000</stddev>
                     </noise>
                 </camera>

File: models/right_camera.xacro (robot description, xacro)
@@ -45,5 +45,5 @@
                         <type>gaussian</type>
                         <mean>0.0</mean>
-                        <stddev>0.007</stddev>
+                        <stddev>0.000</stddev>
                     </noise>
                 </camera>

File: models/turtlebot3_waffle.urdf.xacro (robot description, xacro)
@@ -140,5 +140,5 @@
   <link name="imu_link"/>
   <joint name="camera1_joint" type="fixed">
-    <origin xyz="0 -0.1 0.5" rpy="0 0 0"/>
+    <origin xyz="0 -0.2 0.5" rpy="0 0 0"/>
     <parent link="base_link"/>
     <child link="camera1_link"/>
@@ -146,5 +146,5 @@
   <xacro:left_camera prefix="camera1"/>
   <joint name="camera2_joint" type="fixed">
-    <origin xyz="0.0 0.1 0.5" rpy="0 0 0"/>
+    <origin xyz="0.0 0.2 0.5" rpy="0 0 0"/>
     <parent link="base_link"/>
     <child link="camera2_link"/>

Commit message: finish the line method in real scene.

File: models/left_camera.xacro (robot description, xacro)
@@ -32,5 +32,5 @@
                 <update_rate>30.0</update_rate>
                 <camera name="head">
-                    <horizontal_fov>1.3962634</horizontal_fov>
+                    <horizontal_fov>0.28</horizontal_fov>
                     <image>
                         <width>1280</width>

File: models/right_camera.xacro (robot description, xacro)
@@ -32,5 +32,5 @@
                 <update_rate>30.0</update_rate>
                 <camera name="head">
-                    <horizontal_fov>1.3962634</horizontal_fov>
+                    <horizontal_fov>0.28</horizontal_fov>
                     <image>
                         <width>1280</width>

File: models/turtlebot3_waffle.urdf.xacro (robot description, xacro)
@@ -140,5 +140,5 @@
   <link name="imu_link"/>
   <joint name="camera1_joint" type="fixed">
-    <origin xyz="0 -0.2 0.5" rpy="0 0 0"/>
+    <origin xyz="0 -0.3 1.2" rpy="0 0 0"/>
     <parent link="base_link"/>
     <child link="camera1_link"/>
@@ -146,5 +146,5 @@
   <xacro:left_camera prefix="camera1"/>
   <joint name="camera2_joint" type="fixed">
-    <origin xyz="0.0 0.2 0.5" rpy="0 0 0"/>
+    <origin xyz="0.0 0.3 1.2" rpy="0 0 0"/>
     <parent link="base_link"/>
     <child link="camera2_link"/>
