Commit message: will start to use HoughlinesP

File: models/turtlebot3_waffle.urdf.xacro (robot description, xacro)
@@ -140,5 +140,5 @@
   <link name="imu_link"/>
   <joint name="camera1_joint" type="fixed">
-    <origin xyz="0 -0.3 1.2" rpy="0 0 0"/>
+    <origin xyz="0 0.3 1.2" rpy="0 0 0"/>
     <parent link="base_link"/>
     <child link="camera1_link"/>
@@ -146,5 +146,5 @@
   <xacro:left_camera prefix="camera1"/>
   <joint name="camera2_joint" type="fixed">
-    <origin xyz="0.0 0.3 1.2" rpy="0 0 0"/>
+    <origin xyz="0.0 -0.3 1.2" rpy="0 0 0"/>
     <parent link="base_link"/>
     <child link="camera2_link"/>
